File: schematics/keeby.kicad_pcb (KiCad board)
At the start: 2 copper layers, 139 parts, among them SW1 SW_Push, SW10 SW_Push, SW11 SW_Push, SW12 SW_Push, SW13 SW_Push, SW14 SW_Push, SW15 SW_Push, SW16 SW_Push, SW17 SW_Push, SW18 SW_Push, SW19 SW_Push, SW2 SW_Push, SW20 SW_Push, SW21 SW_Push, SW22 SW_Push, SW23 SW_Push, SW24 SW_Push, SW25 SW_Push, SW26 SW_Push, SW27 SW_Push, SW28 SW_Push, SW29 SW_Push, SW3 SW_Push, SW30 SW_Push, SW31 SW_Push, SW32 SW_Push, SW33 SW_Push, SW34 SW_Push, SW35 SW_Push, SW36 SW_Push, SW37 SW_Push, SW38 SW_Push, SW39 SW_Push, SW4 SW_Push, SW40 SW_Push, SW41 SW_Push, SW42 SW_Push, SW43 SW_Push, SW44 SW_Push, SW45 SW_Push, SW46 SW_Push, SW47 SW_Push, SW48 SW_Push, SW49 SW_Push, SW5 SW_Push, SW50 SW_Push, SW51 SW_Push, SW52 SW_Push, SW53 SW_Push, SW54 SW_Push, SW55 SW_Push, SW56 SW_Push, SW57 SW_Push, SW58 SW_Push, SW59 SW_Push, SW6 SW_Push, SW61 SW_Push, SW63 SW_Push, SW65 SW_Push, SW67 SW_Push, SW68 SW_Push, SW69 SW_Push, SW7 SW_Push, SW70 SW_Push, SW71 SW_Push, SW8 SW_Push, SW9 SW_Push

Commit message: laid out this ratnest is hurting my brain
installed kbplacer to do ts
Parts:
- added D60: 1N4148, Diode_THT:D_DO-35_SOD27_P7.62mm_Horizontal, F.Cu at (73.7, 121.2)
- added D62: 1N4148, Diode_THT:D_DO-35_SOD27_P7.62mm_Horizontal, F.Cu at (168.9, 121.2)
- added D64: 1N4148, Diode_THT:D_DO-35_SOD27_P7.62mm_Horizontal, F.Cu at (257.1, 121.2)
- added D66: 1N4148, Diode_THT:D_DO-35_SOD27_P7.62mm_Horizontal, F.Cu at (295.1, 121.2)
- added D72: 1N4148, Diode_THT:D_DO-35_SOD27_P7.62mm_Horizontal, F.Cu at (255.1, 172.0)
- added D73: 1N4148, Diode_THT:D_DO-35_SOD27_P7.62mm_Horizontal, F.Cu at (255.1, 187.0)
- added D74: 1N4148, Diode_THT:D_DO-35_SOD27_P7.62mm_Horizontal, F.Cu at (255.1, 202.1)
- added D75: 1N4148, Diode_THT:D_DO-35_SOD27_P7.62mm_Horizontal, F.Cu at (255.1, 217.1)
- added D76: SK6812MINI-E, LED_SMD:LED_SK6812MINI-E_3.2x2.8mm_P1.5mm_ReverseMount, F.Cu at (326.6, 159.8)
- added D77: SK6812MINI-E, LED_SMD:LED_SK6812MINI-E_3.2x2.8mm_P1.5mm_ReverseMount, F.Cu at (310.2, 159.2)
- added LED1: SK6812MINI-E, PCM_marbastlib-various:LED_6028R, F.Cu at (297.5, 163.5)
- added SW60: SW_Push, PCM_marbastlib-mx:SW_MX_1u, F.Cu at (64.3, 114.3)
- added SW62: SW_Push, PCM_marbastlib-mx:SW_MX_1u, F.Cu at (159.5, 114.3)
- added SW64: SW_Push, PCM_marbastlib-mx:SW_MX_1u, F.Cu at (247.7, 114.3)
- added SW66: SW_Push, PCM_marbastlib-mx:SW_MX_1u, F.Cu at (285.8, 114.3)
- added SW72: SW_Push, PCM_marbastlib-mx:SW_MX_1u, F.Cu at (245.7, 165.1)
- added SW73: SW_Push, PCM_marbastlib-mx:SW_MX_1u, F.Cu at (245.7, 180.1)
- added SW74: SW_Push, PCM_marbastlib-mx:SW_MX_1u, F.Cu at (245.7, 195.2)
- added SW75: SW_Push, PCM_marbastlib-mx:SW_MX_1u, F.Cu at (245.7, 210.2)
- added SW76: RotaryEncoder_Switch, PCM_marbastlib-various:ROT_Alps_EC11E-Switch, F.Cu at (315.0, 142.5)
- added U1: SuperMini nRF52840, PCM_marbastlib-xp-promicroish:SuperMini_nRF52840_AH_USBup, F.Cu at (239.7, 257.3)
- S3: footprint PCM_marbastlib-mx:STAB_MX_2.25u -> PCM_marbastlib-mx:STAB_MX_6.25u
- moved SW30 287.3 mm to (323.9, 57.1)
- moved SW15 285.4 mm to (323.9, 38.1)
- moved SW29 259.5 mm to (300.0, 57.1)
- moved SW14 254.6 mm to (295.3, 38.1)
- moved SW44 235.0 mm to (323.9, 76.2)
- moved SW28 231.9 mm to (276.2, 57.1)
- moved SW13 224.3 mm to (266.7, 38.1)
- moved SW58 224.0 mm to (323.9, 95.2)
- moved SW10 222.6 mm to (209.6, 38.1)
- moved SW27 209.0 mm to (257.2, 57.1)
- moved SW68 208.2 mm to (323.9, 114.3)
- moved SW43 204.5 mm to (292.9, 76.2)
- moved SW12 204.2 mm to (247.7, 38.1)
- moved SW57 202.8 mm to (304.8, 95.2)
- moved SW9 198.4 mm to (190.5, 38.1)
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- renumbered S4 to S2, S2 to S4
Connections:
- net Net-(A1-GND-Pad13) renamed GND
- A1 pad 11: unconnected-(A1-GPIO8-Pad11) -> /COL3
- A1 pad 12: unconnected-(A1-GPIO9-Pad12) -> /COL4
- A1 pad 14: unconnected-(A1-GPIO10-Pad14) -> /COL5
- A1 pad 15: unconnected-(A1-GPIO11-Pad15) -> /COL6
- A1 pad 16: unconnected-(A1-GPIO12-Pad16) -> /COL7
- A1 pad 17: unconnected-(A1-GPIO13-Pad17) -> /COL8
- A1 pad 19: unconnected-(A1-GPIO14-Pad19) -> /COL9
- A1 pad 20: unconnected-(A1-GPIO15-Pad20) -> /COL10
- A1 pad 21: unconnected-(A1-GPIO16-Pad21) -> /COL11
- A1 pad 22: unconnected-(A1-GPIO17-Pad22) -> /COL12
- A1 pad 24: unconnected-(A1-GPIO18-Pad24) -> /COL13
- A1 pad 25: unconnected-(A1-GPIO19-Pad25) -> /COL13
- A1 pad 26: unconnected-(A1-GPIO20-Pad26) -> /COL14
- A1 pad 27: unconnected-(A1-GPIO21-Pad27) -> /COL15
- A1 pad 36: unconnected-(A1-3V3-Pad36) -> +3V3
- D1 pad 1: /ROW0 -> Net-(D1-K)
- D15 pad 1: /ROW1 -> /ROW0
- D16 pad 1: /ROW1 -> Net-(D1-K)
- D29 pad 1: /ROW3 -> /ROW1
- D30 pad 1: /ROW3 -> /ROW1
- D31 pad 1: /ROW3 -> /ROW1
- D32 pad 1: /ROW3 -> /ROW1
- D43 pad 1: /ROW4 -> /ROW3
- D44 pad 1: /ROW4 -> /ROW3
- D45 pad 1: /ROW4 -> /ROW3
- D46 pad 1: /ROW4 -> /ROW3
- D47 pad 1: /ROW4 -> /ROW3
- D48 pad 1: /ROW4 -> /ROW3
- D57 pad 1: /ROW5 -> /ROW4
- D58 pad 1: /ROW5 -> /ROW4
- D59 pad 1: /ROW5 -> /ROW4
- D61 pad 1: /ROW5 -> /ROW4
- D63 pad 1: /ROW5 -> /ROW4
- SW1 pad 2: Net-(D1-A) -> Net-(D2-A)
- SW10 pad 1: unconnected-(SW10-Pad1) -> /COL9
- SW10 pad 2: Net-(D10-A) -> Net-(D11-A)
- SW11 pad 1: unconnected-(SW11-Pad1) -> /COL10
- SW11 pad 2: Net-(D11-A) -> Net-(D12-A)
- SW12 pad 1: unconnected-(SW12-Pad1) -> /COL11
- SW12 pad 2: Net-(D12-A) -> Net-(D13-A)
- SW13 pad 1: unconnected-(SW13-Pad1) -> /COL12
- SW13 pad 2: Net-(D13-A) -> Net-(D14-A)
- SW14 pad 1: unconnected-(SW14-Pad1) -> /COL13
- SW14 pad 2: Net-(D14-A) -> Net-(D15-A)
- SW15 pad 1: /COL0 -> /COL14
- SW15 pad 2: Net-(D15-A) -> Net-(D1-A)
- SW16 pad 1: /COL1 -> /COL15
- SW17 pad 1: /COL2 -> /COL0
- SW18 pad 1: unconnected-(SW18-Pad1) -> /COL1
- SW19 pad 1: unconnected-(SW19-Pad1) -> /COL2
- SW2 pad 2: Net-(D2-A) -> Net-(D3-A)
- SW20 pad 1: unconnected-(SW20-Pad1) -> /COL3
- SW21 pad 1: unconnected-(SW21-Pad1) -> /COL4
- SW22 pad 1: unconnected-(SW22-Pad1) -> /COL5
- SW23 pad 1: unconnected-(SW23-Pad1) -> /COL6
- SW24 pad 1: unconnected-(SW24-Pad1) -> /COL7
- SW25 pad 1: unconnected-(SW25-Pad1) -> /COL8
- SW26 pad 1: unconnected-(SW26-Pad1) -> /COL9
- SW27 pad 1: unconnected-(SW27-Pad1) -> /COL10
- SW28 pad 1: unconnected-(SW28-Pad1) -> /COL11
- SW29 pad 1: /COL0 -> /COL12
- SW3 pad 2: Net-(D3-A) -> Net-(D4-A)
- SW30 pad 1: /COL1 -> /COL13
- SW31 pad 1: /COL2 -> /COL14
- SW32 pad 1: unconnected-(SW32-Pad1) -> /COL15
- SW33 pad 1: unconnected-(SW33-Pad1) -> /COL0
- SW33 pad 2: Net-(D33-A) -> Net-(D34-A)
- SW34 pad 1: unconnected-(SW34-Pad1) -> /COL1
- SW34 pad 2: Net-(D34-A) -> Net-(D35-A)
- SW35 pad 1: unconnected-(SW35-Pad1) -> /COL2
- SW35 pad 2: Net-(D35-A) -> Net-(D36-A)
- SW36 pad 1: unconnected-(SW36-Pad1) -> /COL3
- SW36 pad 2: Net-(D36-A) -> Net-(D37-A)
- SW37 pad 1: unconnected-(SW37-Pad1) -> /COL4
- SW37 pad 2: Net-(D37-A) -> Net-(D38-A)
- SW38 pad 1: unconnected-(SW38-Pad1) -> /COL5
- SW38 pad 2: Net-(D38-A) -> Net-(D39-A)
- SW39 pad 1: unconnected-(SW39-Pad1) -> /COL6
- SW39 pad 2: Net-(D39-A) -> Net-(D40-A)
- SW4 pad 1: unconnected-(SW4-Pad1) -> /COL3
- SW4 pad 2: Net-(D4-A) -> Net-(D5-A)
- SW40 pad 1: unconnected-(SW40-Pad1) -> /COL7
- SW40 pad 2: Net-(D40-A) -> Net-(D41-A)
- SW41 pad 1: unconnected-(SW41-Pad1) -> /COL8
- SW41 pad 2: Net-(D41-A) -> Net-(D42-A)
- SW42 pad 1: unconnected-(SW42-Pad1) -> /COL9
- SW42 pad 2: Net-(D42-A) -> Net-(D43-A)
- SW43 pad 1: /COL0 -> /COL10
- SW43 pad 2: Net-(D43-A) -> Net-(D44-A)
- SW44 pad 1: /COL1 -> /COL11
- SW44 pad 2: Net-(D44-A) -> Net-(D45-A)
- SW45 pad 1: /COL2 -> /COL12
- SW45 pad 2: Net-(D45-A) -> Net-(D46-A)
- SW46 pad 1: unconnected-(SW46-Pad1) -> /COL13
- SW46 pad 2: Net-(D46-A) -> Net-(D47-A)
- SW47 pad 1: unconnected-(SW47-Pad1) -> /COL14
- SW47 pad 2: Net-(D47-A) -> Net-(D33-A)
- SW48 pad 1: unconnected-(SW48-Pad1) -> /COL15
- SW49 pad 1: unconnected-(SW49-Pad1) -> /COL0
- SW5 pad 1: unconnected-(SW5-Pad1) -> /COL4
- SW5 pad 2: Net-(D5-A) -> Net-(D6-A)
- SW50 pad 1: unconnected-(SW50-Pad1) -> /COL1
- SW51 pad 1: unconnected-(SW51-Pad1) -> /COL2
- SW52 pad 1: unconnected-(SW52-Pad1) -> /COL3
- SW53 pad 1: unconnected-(SW53-Pad1) -> /COL4
- SW54 pad 1: unconnected-(SW54-Pad1) -> /COL5
- SW55 pad 1: unconnected-(SW55-Pad1) -> /COL6
- SW56 pad 1: unconnected-(SW56-Pad1) -> /COL7
- SW57 pad 1: /COL0 -> /COL8
- SW58 pad 1: /COL1 -> /COL9
- SW59 pad 1: /COL2 -> /COL10
- SW6 pad 1: unconnected-(SW6-Pad1) -> /COL5
- SW6 pad 2: Net-(D6-A) -> Net-(D7-A)
- SW61 pad 1: unconnected-(SW61-Pad1) -> /COL12
- SW63 pad 1: unconnected-(SW63-Pad1) -> /COL14
- SW65 pad 1: unconnected-(SW65-Pad1) -> /COL0
- SW67 pad 1: unconnected-(SW67-Pad1) -> /COL2
- SW68 pad 1: unconnected-(SW68-Pad1) -> /COL4
- SW69 pad 1: unconnected-(SW69-Pad1) -> /COL9
- SW7 pad 1: unconnected-(SW7-Pad1) -> /COL6
- SW7 pad 2: Net-(D7-A) -> Net-(D8-A)
- SW70 pad 1: unconnected-(SW70-Pad1) -> /COL10
- SW71 pad 1: unconnected-(SW71-Pad1) -> /COL11
- SW8 pad 1: unconnected-(SW8-Pad1) -> /COL7
- SW8 pad 2: Net-(D8-A) -> Net-(D9-A)
- SW9 pad 1: unconnected-(SW9-Pad1) -> /COL8
- SW9 pad 2: Net-(D9-A) -> Net-(D10-A)
Other:
- board outline added: 365.3 x 208.6 mm

Commit message: I have narrowed down the headache of all the keys. I can route peacefully now.
+maybe some uncommitted changes from a few days ago as well...
Parts:
- removed D71, D72, D73, D74, D75: 1N4148, Diode_THT:D_DO-35_SOD27_P7.62mm_Horizontal
- removed D76, D77: SK6812MINI-E, LED_SMD:LED_SK6812MINI-E_3.2x2.8mm_P1.5mm_ReverseMount
- removed SW72, SW73, SW74, SW75: SW_Push, PCM_marbastlib-mx:SW_MX_1u
- removed SW76: RotaryEncoder_Switch, PCM_marbastlib-various:ROT_Alps_EC11E-Switch
- added LED2: SK6812MINI-E, LED_SMD:LED_SK6812MINI-E_3.2x2.8mm_P1.5mm_ReverseMount, F.Cu at (273.1, 172.8)
- added LED3: SK6812MINI-E, PCM_marbastlib-various:LED_6028R, F.Cu at (362.9, 168.7)
- LED1: footprint PCM_marbastlib-various:LED_6028R -> LED_SMD:LED_SK6812MINI-E_3.2x2.8mm_P1.5mm_ReverseMount
- S2: footprint PCM_marbastlib-mx:STAB_MX_2.25u -> PCM_marbastlib-mx:STAB_MX_6.25u
- S3: footprint PCM_marbastlib-mx:STAB_MX_6.25u -> PCM_marbastlib-mx:STAB_MX_2.25u
- SW69: value SW_Push -> RotaryEncoder_Switch; footprint PCM_marbastlib-mx:SW_MX_1u -> PCM_marbastlib-various:ROT_Alps_EC11E-Switch
- moved D31 275.9 mm to (330.5, 81.0), turned to 180 degrees
- moved S1 257.8 mm to (295.3, 15.7)
- moved D46 180.6 mm to (240.0, 100.0), turned to 180 degrees
- moved S4 173.6 mm to (292.9, 76.2)
- moved SW71 151.7 mm to (350.8, 259.5)
- moved D69 148.4 mm to (357.5, 249.2)
- moved D70 148.4 mm to (357.5, 264.2)
- moved SW70 143.2 mm to (350.8, 244.4)
- moved S2 138.7 mm to (159.5, 114.3)
- moved D45 132.4 mm to (201.9, 100.0), turned to 180 degrees
- moved S3 111.2 mm to (50.0, 95.2)
- moved D62 104.4 mm to (273.3, 119.0), turned to 180 degrees
- moved LED1 76.6 mm to (234.8, 207.5), turned to 90 degrees
- moved D63 71.9 mm to (166.2, 119.0), turned to 180 degrees
- moved SW69 61.6 mm to (173.7, 175.0)
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Connections:
- D1 pad 1: Net-(D1-K) -> /ROW0
- D16 pad 1: Net-(D1-K) -> /ROW1
- D31 pad 1: /ROW1 -> /ROW3
- D32 pad 1: /ROW1 -> /ROW3
- D45 pad 1: /ROW3 -> /ROW4
- D46 pad 1: /ROW3 -> /ROW4
- D47 pad 1: /ROW3 -> /ROW4
- D48 pad 1: /ROW3 -> /ROW4
- D59 pad 1: /ROW4 -> /ROW5
- D60 pad 1: /ROW4 -> /ROW5
- D61 pad 1: /ROW4 -> /ROW5
- D62 pad 1: /ROW4 -> /ROW5
- D63 pad 1: /ROW4 -> /ROW5
- D64 pad 1: /ROW4 -> /ROW5
- D69 pad 1: /ROW5 -> unconnected-(D69-K-Pad1)
- D70 pad 1: /ROW5 -> unconnected-(D70-K-Pad1)
- LED1 pad 1: unconnected-(LED1-VDD-Pad1) -> GND
- LED1 pad 3: unconnected-(LED1-DIN-Pad3) -> +3V3
- LED1 pad 4: unconnected-(LED1-VSS-Pad4) -> Net-(LED1-DOUT)
- SW16 pad 1: /COL15 -> /COL0
- SW17 pad 1: /COL0 -> /COL1
- SW18 pad 1: /COL1 -> /COL2
- SW19 pad 1: /COL2 -> /COL3
- SW20 pad 1: /COL3 -> /COL4
- SW21 pad 1: /COL4 -> /COL5
- SW22 pad 1: /COL5 -> /COL6
- SW23 pad 1: /COL6 -> /COL7
- SW24 pad 1: /COL7 -> /COL8
- SW25 pad 1: /COL8 -> /COL9
- SW26 pad 1: /COL9 -> /COL10
- SW27 pad 1: /COL10 -> /COL11
- SW28 pad 1: /COL11 -> /COL12
- SW29 pad 1: /COL12 -> /COL13
- SW30 pad 1: /COL13 -> /COL14
- SW31 pad 1: /COL14 -> /COL0
- SW31 pad 2: Net-(D31-A) -> Net-(D32-A)
- SW32 pad 1: /COL15 -> /COL1
- SW32 pad 2: Net-(D32-A) -> Net-(D33-A)
- SW33 pad 1: /COL0 -> /COL2
- SW34 pad 1: /COL1 -> /COL3
- SW35 pad 1: /COL2 -> /COL4
- SW36 pad 1: /COL3 -> /COL5
- SW37 pad 1: /COL4 -> /COL6
- SW38 pad 1: /COL5 -> /COL7
- SW39 pad 1: /COL6 -> /COL8
- SW40 pad 1: /COL7 -> /COL9
- SW41 pad 1: /COL8 -> /COL10
- SW42 pad 1: /COL9 -> /COL11
- SW43 pad 1: /COL10 -> /COL13
- SW44 pad 1: /COL11 -> /COL14
- SW44 pad 2: Net-(D45-A) -> Net-(D31-A)
- SW45 pad 1: /COL12 -> /COL0
- SW45 pad 2: Net-(D46-A) -> Net-(D47-A)
- SW46 pad 1: /COL13 -> /COL1
- SW46 pad 2: Net-(D47-A) -> Net-(D48-A)
- SW47 pad 1: /COL14 -> /COL2
- SW47 pad 2: Net-(D33-A) -> Net-(D49-A)
- SW48 pad 1: /COL15 -> /COL3
- SW48 pad 2: Net-(D48-A) -> Net-(D50-A)
- SW49 pad 1: /COL0 -> /COL4
- SW49 pad 2: Net-(D49-A) -> Net-(D51-A)
- SW50 pad 1: /COL1 -> /COL5
- SW50 pad 2: Net-(D50-A) -> Net-(D52-A)
- SW51 pad 1: /COL2 -> /COL6
- SW51 pad 2: Net-(D51-A) -> Net-(D53-A)
- SW52 pad 1: /COL3 -> /COL7
- SW52 pad 2: Net-(D52-A) -> Net-(D45-A)
- SW53 pad 1: /COL4 -> /COL8
- SW53 pad 2: Net-(D53-A) -> Net-(D54-A)
- SW54 pad 1: /COL5 -> /COL9
- SW54 pad 2: Net-(D54-A) -> Net-(D46-A)
- SW55 pad 1: /COL6 -> /COL10
- SW56 pad 1: /COL7 -> /COL12
- SW57 pad 1: /COL8 -> /COL13
- SW58 pad 1: /COL9 -> /COL14
- SW59 pad 1: /COL10 -> /COL0
- SW60 pad 1: /COL11 -> /COL1
- SW61 pad 1: /COL12 -> /COL2
- SW62 pad 1: /COL13 -> /COL8
- SW62 pad 2: Net-(D62-A) -> Net-(D63-A)
- SW63 pad 1: /COL14 -> /COL9
- SW63 pad 2: Net-(D63-A) -> Net-(D64-A)
- SW64 pad 1: /COL15 -> /COL10
- SW64 pad 2: Net-(D64-A) -> Net-(D65-A)
- SW65 pad 1: /COL0 -> /COL5
- SW65 pad 2: Net-(D65-A) -> Net-(D62-A)
- SW66 pad 1: /COL1 -> /COL12
- SW67 pad 1: /COL2 -> /COL13
- SW68 pad 1: /COL4 -> /COL14
- SW70 pad 1: /COL10 -> unconnected-(SW70-Pad1)
- SW70 pad 2: Net-(D70-A) -> Net-(D69-A)
- SW71 pad 1: /COL11 -> unconnected-(SW71-Pad1)
- SW71 pad 2: Net-(D71-A) -> Net-(D70-A)
Other:
- board size 365.3 x 208.6 mm -> 355.7 x 208.6 mm

Commit message: more hours of work
Parts:
- removed D69, D70: 1N4148, Diode_THT:D_DO-35_SOD27_P7.62mm_Horizontal
- removed LED3: SK6812MINI-E, PCM_marbastlib-various:LED_6028R
- removed SW70, SW71: SW_Push, PCM_marbastlib-mx:SW_MX_1u
- added REF**: joystick_psp1000, PCM_marbastlib-xp-various:PNT_psp1000, F.Cu at (346.0, 90.0)
- S2: renamed from S1; footprint PCM_marbastlib-mx:STAB_MX_2.25u -> PCM_marbastlib-mx:STAB_MX_2u
- moved SW16 182.5 mm to (345.0, 112.0), turned to 180 degrees
- moved LED1 139.7 mm to (347.0, 124.3), turned to 0 degrees
- moved U1 107.4 mm to (249.6, 150.3)
- moved SW66 107.2 mm to (159.5, 114.3)
- moved D62 105.6 mm to (167.7, 121.5), turned to 90 degrees
- moved LED2 81.0 mm to (338.3, 124.8)
- moved D63 70.7 mm to (236.8, 121.5), turned to 90 degrees
- moved SW63 69.1 mm to (228.6, 114.3)
- moved S2 22.4 mm to (295.3, 38.1)
- moved D64 20.8 mm to (255.8, 121.5), turned to 90 degrees
- moved D65 20.8 mm to (274.9, 121.5), turned to 90 degrees
- moved SW64 19.1 mm to (247.7, 114.3)
- moved SW65 19.0 mm to (266.7, 114.3)
- moved D19 2.94 mm to (113.0, 64.4), turned to 90 degrees
- moved D21 2.94 mm to (151.1, 64.4), turned to 90 degrees
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- renumbered S4 to S1, S2 to S4, SW69 to SW16, SW16 to SW17, SW17 to SW18, SW18 to SW19, SW19 to SW20, SW20 to SW21, SW21 to SW22, SW22 to SW23, SW23 to SW24, SW24 to SW25, SW25 to SW26, SW26 to SW27, SW27 to SW28, SW28 to SW29, SW29 to SW30, SW30 to SW31, SW31 to SW32, SW32 to SW33, SW33 to SW34, SW34 to SW35, SW35 to SW36, SW36 to SW37, SW37 to SW38, SW38 to SW39, SW39 to SW40, SW40 to SW41, SW41 to SW42, SW42 to SW43, SW43 to SW44, SW44 to SW45, SW45 to SW46, SW46 to SW47, SW47 to SW48, SW48 to SW49, SW49 to SW50, SW50 to SW51, SW51 to SW52, SW52 to SW53, SW53 to SW54, SW54 to SW55, SW55 to SW56, SW56 to SW57, SW57 to SW58, SW58 to SW59, SW59 to SW60, SW60 to SW61, SW61 to SW62, SW62 to SW63, SW63 to SW64, SW64 to SW65, SW65 to SW66, SW66 to SW67, SW67 to SW68, SW68 to SW69
Connections:
- A1 pad 25: /COL13 -> /COL14
- A1 pad 26: /COL14 -> unconnected-(A1-GPIO20-Pad26)
- A1 pad 27: /COL15 -> unconnected-(A1-GPIO21-Pad27)
Routing:
- net /COL8: track 0.00 -> 310.4 mm
- net /ROW0: track 0.00 -> 285.8 mm
- net /ROW5: track 0.00 -> 285.6 mm
- net /ROW1: track 0.00 -> 281.0 mm
- net /ROW3: track 0.00 -> 280.8 mm
- net /ROW4: track 0.00 -> 275.0 mm
- net /COL14: track 0.00 -> 123.5 mm
- net /COL1: track 0.00 -> 93.6 mm
- net /COL9: track 0.00 -> 92.0 mm
- net /COL10: track 0.00 -> 92.0 mm
- net /COL2: track 0.00 -> 91.0 mm
- net /COL5: track 0.00 -> 87.0 mm
- net /COL13: track 0.00 -> 86.1 mm
- net /COL0: track 0.00 -> 85.8 mm
- net /COL12: track 0.00 -> 84.1 mm
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- added copper zone on B.Cu, net GND
Other:
- board size 355.7 x 208.6 mm -> 335 x 105 mm

Commit message: checkpointer. readme stuff. more journal. fix switch order
Parts:
- removed REF**: joystick_psp1000, PCM_marbastlib-xp-various:PNT_psp1000
- added JS1: joystick_analog, PCM_marbastlib-xp-various:PNT_psp1000, F.Cu at (346.0, 90.0)
- moved D65 107.2 mm to (274.9, 121.5)
- moved SW65 107.2 mm to (266.7, 114.3)
- moved D62 69.1 mm to (167.7, 121.5)
- moved SW62 69.1 mm to (159.5, 114.3)
- moved D63 19.1 mm to (236.8, 121.5)
- moved SW63 19.1 mm to (228.6, 114.3)
- moved D64 19.0 mm to (255.8, 121.5)
- moved SW64 19.0 mm to (247.7, 114.3)
- renumbered D2 to D1, D11 to D10, D12 to D11, D13 to D12, D14 to D13, D15 to D14, D1 to D15, D3 to D2, D4 to D3, D32 to D31, D33 to D32, D34 to D33, D35 to D34, D36 to D35, D37 to D36, D38 to D37, D39 to D38, D40 to D39, D5 to D4, D41 to D40, D42 to D41, D43 to D42, D44 to D43, D31 to D44, D6 to D5, D7 to D6, D63 to D62, D64 to D63, D65 to D64, D62 to D65, D8 to D7, D9 to D8, D10 to D9, SW16 to EC1, SW17 to SW16, SW18 to SW17, SW19 to SW18, SW20 to SW19, SW21 to SW20, SW22 to SW21, SW23 to SW22, SW24 to SW23, SW25 to SW24, SW26 to SW25, SW27 to SW26, SW28 to SW27, SW29 to SW28, SW30 to SW29, SW31 to SW30, SW32 to SW31, SW33 to SW32, SW34 to SW33, SW35 to SW34, SW36 to SW35, SW37 to SW36, SW38 to SW37, SW39 to SW38, SW40 to SW39, SW41 to SW40, SW42 to SW41, SW43 to SW42, SW44 to SW43, SW45 to SW44, SW46 to SW45, SW47 to SW46, SW48 to SW47, SW49 to SW48, SW50 to SW49, SW51 to SW50, SW52 to SW51, SW53 to SW52, SW54 to SW53, SW55 to SW54, SW56 to SW55, SW57 to SW56, SW58 to SW57, SW59 to SW58, SW60 to SW59, SW61 to SW60, SW62 to SW61, SW63 to SW62, SW64 to SW63, SW65 to SW64, SW66 to SW65, SW67 to SW66, SW68 to SW67, SW69 to SW68
Connections:
- SW62 pad 1: /COL8 -> /COL5
- SW63 pad 1: /COL9 -> /COL8
- SW64 pad 1: /COL10 -> /COL9
- SW65 pad 1: /COL5 -> /COL10

Commit message: connected the nrf to the column/rows.
Parts:
- added U2: MCP23017x-x-SP, Package_DIP:DIP-28_W7.62mm, F.Cu at (269.2, 134.5)
- moved U1 147.6 mm to (346.3, 38.8)
- moved A1 140.6 mm to (290.2, 159.5)
- moved LED1 5.01 mm to (352.0, 124.0)
- moved JS1 5.00 mm to (346.0, 85.0)
- moved LED2 3.36 mm to (341.6, 124.0)
Connections:
- A1 pad 1: /ROW0 -> unconnected-(A1-GPIO0-Pad1)
- A1 pad 10: /COL2 -> unconnected-(A1-GPIO7-Pad10)
- A1 pad 11: /COL3 -> unconnected-(A1-GPIO8-Pad11)
- A1 pad 12: /COL4 -> unconnected-(A1-GPIO9-Pad12)
- A1 pad 13: GND -> Net-(A1-GND-Pad13)
- A1 pad 14: /COL5 -> unconnected-(A1-GPIO10-Pad14)
- A1 pad 15: /COL6 -> unconnected-(A1-GPIO11-Pad15)
- A1 pad 16: /COL7 -> unconnected-(A1-GPIO12-Pad16)
- A1 pad 17: /COL8 -> unconnected-(A1-GPIO13-Pad17)
- A1 pad 18: GND -> Net-(A1-GND-Pad13)
- A1 pad 19: /COL9 -> unconnected-(A1-GPIO14-Pad19)
- A1 pad 2: /ROW1 -> unconnected-(A1-GPIO1-Pad2)
- A1 pad 20: /COL10 -> unconnected-(A1-GPIO15-Pad20)
- A1 pad 21: /COL11 -> unconnected-(A1-GPIO16-Pad21)
- A1 pad 22: /COL12 -> unconnected-(A1-GPIO17-Pad22)
- A1 pad 23: GND -> Net-(A1-GND-Pad13)
- A1 pad 24: /COL13 -> unconnected-(A1-GPIO18-Pad24)
- A1 pad 25: /COL14 -> unconnected-(A1-GPIO19-Pad25)
- A1 pad 28: GND -> Net-(A1-GND-Pad13)
- A1 pad 3: GND -> Net-(A1-GND-Pad13)
- A1 pad 36: +3V3 -> unconnected-(A1-3V3-Pad36)
- A1 pad 38: GND -> Net-(A1-GND-Pad13)
- A1 pad 4: /ROW3 -> unconnected-(A1-GPIO2-Pad4)
- A1 pad 5: /ROW4 -> unconnected-(A1-GPIO3-Pad5)
- A1 pad 6: /ROW5 -> unconnected-(A1-GPIO4-Pad6)
- A1 pad 7: /COL0 -> unconnected-(A1-GPIO5-Pad7)
- A1 pad 8: GND -> Net-(A1-GND-Pad13)
- A1 pad 9: /COL1 -> unconnected-(A1-GPIO6-Pad9)
- U1 pad 1: unconnected-(U1-P0.06-Pad1) -> /ROW0
- U1 pad 10: unconnected-(U1-P0.11-Pad10) -> /COL2
- U1 pad 11: unconnected-(U1-P1.04-LF-Pad11) -> /COL3
- U1 pad 12: unconnected-(U1-P1.06-LF-Pad12) -> /COL4
- U1 pad 14: unconnected-(U1-GND-Pad14) -> GND
- U1 pad 15: unconnected-(U1-RST-Pad15) -> +3V3
- U1 pad 17: unconnected-(U1-P0.31-LF-Pad17) -> /COL5
- U1 pad 18: unconnected-(U1-P0.29-LF-Pad18) -> /COL6
- U1 pad 19: unconnected-(U1-P0.02-LF-Pad19) -> /COL7
- U1 pad 2: unconnected-(U1-P0.08-Pad2) -> /ROW1
- U1 pad 20: unconnected-(U1-P1.15-LF-Pad20) -> /COL8
- U1 pad 21: unconnected-(U1-P1.13-LF-Pad21) -> /COL9
- U1 pad 22: unconnected-(U1-P1.11-LF-Pad22) -> /COL10
- U1 pad 23: unconnected-(U1-P0.10-LF-Pad23) -> /COL11
- U1 pad 24: unconnected-(U1-P0.09-LF-Pad24) -> /COL12
- U1 pad 26: unconnected-(U1-P1.02-LF-Pad26) -> /COL14
- U1 pad 27: unconnected-(U1-P1.07-LF-Pad27) -> /COL13
- U1 pad 28: unconnected-(U1-GND-Pad28) -> GND
- U1 pad 3: unconnected-(U1-GND-Pad3) -> GND
- U1 pad 4: unconnected-(U1-GND-Pad4) -> GND
- U1 pad 5: unconnected-(U1-P0.17-Pad5) -> /ROW3
- U1 pad 6: unconnected-(U1-P0.20-Pad6) -> /ROW4
- U1 pad 7: unconnected-(U1-P0.22-Pad7) -> /ROW5
- U1 pad 8: unconnected-(U1-P0.24-Pad8) -> /COL0
- U1 pad 9: unconnected-(U1-P1.00-Pad9) -> /COL1
Routing:
- net /COL8: track 310.4 -> 103.9 mm
- net /COL14: track 123.5 -> 76.2 mm
Other:
- board size 335 x 105 mm -> 329.4 x 105 mm

Commit message: added nrf 3d models and all the other needed models
models and nrf
the commit before had a few things merged together that I actually wanted to separate into different commits
Parts:
- added H1: MountingHole, MountingHole:MountingHole_2.1mm, F.Cu at (30.5, 26.0)
- added H2: MountingHole, MountingHole:MountingHole_2.1mm, F.Cu at (328.5, 26.0)
- added H3: MountingHole, MountingHole:MountingHole_2.1mm, F.Cu at (30.5, 126.2)
- added H4: MountingHole, MountingHole:MountingHole_2.1mm, F.Cu at (328.5, 126.2)
- LED1, LED2: moved to B.Cu
- moved U2 143.1 mm to (358.5, 22.6)
- moved EC1 3.52 mm to (345.4, 115.5), turned to -90 degrees
- moved LED1 3.02 mm to (350.8, 126.8), turned to 180 degrees
- moved LED2 2.75 mm to (341.6, 126.8), turned to 180 degrees
- moved U1 1.93 mm to (346.3, 40.8)
Routing:
- net GND: track 0.00 -> 15.5 mm
- net /COL8: track 103.9 -> 94.7 mm
Other:
- board size 329.4 x 105 mm -> 329.4 x 105.9 mm
