File: schematics/keeby.kicad_pcb (KiCad board)
At the start: 2 copper layers, 329.4 x 105.9 mm, 151 parts, among them SW1 SW_Push, SW10 SW_Push, SW11 SW_Push, SW12 SW_Push, SW13 SW_Push, SW14 SW_Push, SW15 SW_Push, SW16 SW_Push, SW17 SW_Push, SW18 SW_Push, SW19 SW_Push, SW2 SW_Push, SW20 SW_Push, SW21 SW_Push, SW22 SW_Push, SW23 SW_Push, SW24 SW_Push, SW25 SW_Push, SW26 SW_Push, SW27 SW_Push, SW28 SW_Push, SW29 SW_Push, SW3 SW_Push, SW30 SW_Push, SW31 SW_Push, SW32 SW_Push, SW33 SW_Push, SW34 SW_Push, SW35 SW_Push, SW36 SW_Push, SW37 SW_Push, SW38 SW_Push, SW39 SW_Push, SW4 SW_Push, SW40 SW_Push, SW41 SW_Push, SW42 SW_Push, SW43 SW_Push, SW44 SW_Push, SW45 SW_Push, SW46 SW_Push, SW47 SW_Push, SW48 SW_Push, SW49 SW_Push, SW5 SW_Push, SW50 SW_Push, SW51 SW_Push, SW52 SW_Push, SW53 SW_Push, SW54 SW_Push, SW55 SW_Push, SW56 SW_Push, SW57 SW_Push, SW58 SW_Push, SW59 SW_Push, SW6 SW_Push, SW60 SW_Push, SW61 SW_Push, SW62 SW_Push, SW63 SW_Push, SW64 SW_Push, SW65 SW_Push, SW66 SW_Push, SW67 SW_Push, SW68 SW_Push, SW7 SW_Push, SW8 SW_Push, SW9 SW_Push, U1 SuperMini nRF52840, U2 MCP23017x-x-SP

Commit message: help
Parts:
- removed A1: RaspberryPi_Pico, Module:RaspberryPi_Pico_Common_THT
- added G***: LOGO, LOGO, B.Cu at (103.2, 127.5)
- H1, H2, H3, H4: footprint MountingHole:MountingHole_2.1mm -> MountingHole:MountingHole_2.2mm_M2
- moved JS1 301.5 mm to (47.0, 46.3), turned to -90 degrees
- moved EC1 282.5 mm to (71.8, 45.3)
- moved LED1 95.4 mm to (296.1, 48.5)
- moved LED2 86.0 mm to (296.1, 53.8)
- moved U2 77.2 mm to (283.8, 41.8), turned to -90 degrees
- moved H2 39.7 mm to (291.2, 39.7)
- moved D59 27.5 mm to (48.7, 149.1)
- moved D60 27.5 mm to (72.5, 149.1)
- moved D61 27.5 mm to (96.3, 149.1)
- moved D62 27.5 mm to (167.7, 149.1)
- moved D63 27.5 mm to (236.8, 149.1)
- moved D64 27.5 mm to (255.8, 149.1)
- moved D65 27.5 mm to (274.9, 149.1)
- moved D66 27.5 mm to (293.9, 149.1)
- moved D67 27.5 mm to (313.0, 149.1)
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Connections:
- JS1 pad 1: unconnected-(JS1-X-Pad1) -> /A1
- JS1 pad 3: unconnected-(JS1-Y-Pad3) -> /A0
- U2 pad 12: unconnected-(U2-SCK-Pad12) -> /SCL
- U2 pad 13: unconnected-(U2-SDA-Pad13) -> /SDA
Routing:
- net GND: track 15.5 -> 10.1 mm
Other:
- board size 329.4 x 105.9 mm -> 315 x 119.5 mm
- board text added: "THE KAI BOARD"

Commit message: a bunch of messy routing and wiring
Parts:
- added G***: LOGO, LOGO, F.Cu at (158.2, 87.8)
- added G***: LOGO, LOGO, B.Cu at (276.6, 111.7)
- added REF**: SW_MSK12C02-HB, PCM_marbastlib-various:SW_MSK12C02-HB, F.Cu at (371.5, 55.0)
- moved JS1 24.6 mm to (71.6, 46.4)
- moved EC1 22.5 mm to (49.4, 47.9), turned to 90 degrees
- moved U1 1.10 mm to (321.7, 44.8)
- moved H4 0.48 mm to (336.5, 152.0)
Connections:
- D1 pad 1: /ROW0 -> /ROW1
- D10 pad 1: /ROW0 -> /ROW1
- D11 pad 1: /ROW0 -> /ROW1
- D12 pad 1: /ROW0 -> /ROW1
- D13 pad 1: /ROW0 -> /ROW1
- D14 pad 1: /ROW0 -> /ROW1
- D15 pad 1: /ROW0 -> /ROW1
- D16 pad 1: /ROW1 -> /ROW2
- D17 pad 1: /ROW1 -> /ROW2
- D18 pad 1: /ROW1 -> /ROW2
- D19 pad 1: /ROW1 -> /ROW2
- D2 pad 1: /ROW0 -> /ROW1
- D20 pad 1: /ROW1 -> /ROW2
- D21 pad 1: /ROW1 -> /ROW2
- D22 pad 1: /ROW1 -> /ROW2
- D23 pad 1: /ROW1 -> /ROW2
- D24 pad 1: /ROW1 -> /ROW2
- D25 pad 1: /ROW1 -> /ROW2
- D26 pad 1: /ROW1 -> /ROW2
- D27 pad 1: /ROW1 -> /ROW2
- D28 pad 1: /ROW1 -> /ROW2
- D29 pad 1: /ROW1 -> /ROW2
- D3 pad 1: /ROW0 -> /ROW1
- D30 pad 1: /ROW1 -> /ROW2
- D4 pad 1: /ROW0 -> /ROW1
- D5 pad 1: /ROW0 -> /ROW1
- D6 pad 1: /ROW0 -> /ROW1
- D7 pad 1: /ROW0 -> /ROW1
- D8 pad 1: /ROW0 -> /ROW1
- D9 pad 1: /ROW0 -> /ROW1
- EC1 pad A: unconnected-(EC1-PadA) -> Net-(U2-GPB1)
- EC1 pad B: unconnected-(EC1-PadB) -> Net-(U2-GPB2)
- EC1 pad S2: unconnected-(EC1-PadS2) -> Net-(U2-GPB0)
- SW1 pad 1: /COL0 -> /COL1
- SW10 pad 1: /COL9 -> /COL10
- SW11 pad 1: /COL10 -> /COL11
- SW12 pad 1: /COL11 -> /COL12
- SW13 pad 1: /COL12 -> /COL13
- SW14 pad 1: /COL13 -> /COL14
- SW15 pad 1: /COL14 -> /COL15
- SW16 pad 1: /COL0 -> /COL1
- SW17 pad 1: /COL1 -> /COL2
- SW18 pad 1: /COL2 -> /COL3
- SW19 pad 1: /COL3 -> /COL4
- SW2 pad 1: /COL1 -> /COL2
- SW20 pad 1: /COL4 -> /COL5
- SW21 pad 1: /COL5 -> /COL6
- SW22 pad 1: /COL6 -> /COL7
- SW23 pad 1: /COL7 -> /COL8
- SW24 pad 1: /COL8 -> /COL9
- SW25 pad 1: /COL9 -> /COL10
- SW26 pad 1: /COL10 -> /COL11
- SW27 pad 1: /COL11 -> /COL12
- SW28 pad 1: /COL12 -> /COL13
- SW29 pad 1: /COL13 -> /COL14
- SW3 pad 1: /COL2 -> /COL3
- SW30 pad 1: /COL14 -> /COL15
- SW31 pad 1: /COL0 -> /COL1
- SW32 pad 1: /COL1 -> /COL2
- SW33 pad 1: /COL2 -> /COL3
- SW34 pad 1: /COL3 -> /COL4
- SW35 pad 1: /COL4 -> /COL5
- SW36 pad 1: /COL5 -> /COL6
- SW37 pad 1: /COL6 -> /COL7
- SW38 pad 1: /COL7 -> /COL8
- SW39 pad 1: /COL8 -> /COL9
- SW4 pad 1: /COL3 -> /COL4
- SW40 pad 1: /COL9 -> /COL10
- SW41 pad 1: /COL10 -> /COL11
- SW42 pad 1: /COL11 -> /COL12
- SW43 pad 1: /COL13 -> /COL14
- SW44 pad 1: /COL14 -> /COL15
- SW45 pad 1: /COL0 -> /COL1
- SW46 pad 1: /COL1 -> /COL2
- SW47 pad 1: /COL2 -> /COL3
- SW48 pad 1: /COL3 -> /COL4
- SW49 pad 1: /COL4 -> /COL5
- SW5 pad 1: /COL4 -> /COL5
- SW50 pad 1: /COL5 -> /COL6
- SW51 pad 1: /COL6 -> /COL7
- SW52 pad 1: /COL7 -> /COL8
- SW53 pad 1: /COL8 -> /COL9
- SW54 pad 1: /COL9 -> /COL10
- SW55 pad 1: /COL10 -> /COL11
- SW56 pad 1: /COL12 -> /COL13
- SW57 pad 1: /COL13 -> /COL14
- SW58 pad 1: /COL14 -> /COL15
- SW59 pad 1: /COL0 -> /COL1
- SW6 pad 1: /COL5 -> /COL6
- SW60 pad 1: /COL1 -> /COL2
- SW61 pad 1: /COL2 -> /COL3
- SW62 pad 1: /COL5 -> /COL6
- SW63 pad 1: /COL8 -> /COL9
- SW64 pad 1: /COL9 -> /COL10
- SW65 pad 1: /COL10 -> /COL11
- SW66 pad 1: /COL12 -> /COL13
- SW67 pad 1: /COL13 -> /COL14
- SW68 pad 1: /COL14 -> /COL15
- SW7 pad 1: /COL6 -> /COL7
- SW8 pad 1: /COL7 -> /COL8
- SW9 pad 1: /COL8 -> /COL9
- U1 pad 1: /ROW0 -> /COL1
- U1 pad 10: /COL2 -> /COL8
- U1 pad 11: /COL3 -> /COL9
- U1 pad 12: /COL4 -> /COL10
- U1 pad 15: +3V3 -> unconnected-(U1-RST-Pad15)
- U1 pad 16: unconnected-(U1-3V3-Pad16) -> +3V3
- U1 pad 17: /COL5 -> /ROW5
- U1 pad 18: /COL6 -> /ROW4
- U1 pad 19: /COL7 -> /ROW3
- U1 pad 2: /ROW1 -> /COL2
- U1 pad 20: /COL8 -> /ROW2
- U1 pad 21: /COL9 -> /ROW1
- U1 pad 22: /COL10 -> /COL13
- U1 pad 23: /COL11 -> /COL12
- U1 pad 24: /COL12 -> /COL11
- U1 pad 26: /COL14 -> /COL15
- U1 pad 27: /COL13 -> /COL14
- U1 pad 5: /ROW3 -> /COL3
- U1 pad 6: /ROW4 -> /COL4
- U1 pad 7: /ROW5 -> /COL5
- U1 pad 8: /COL0 -> /COL6
- U1 pad 9: /COL1 -> /COL7
- U2 pad 1: unconnected-(U2-GPB0-Pad1) -> Net-(U2-GPB0)
- U2 pad 10: unconnected-(U2-V_{SS}-Pad10) -> GND
- U2 pad 15: unconnected-(U2-A0-Pad15) -> /A0
- U2 pad 16: unconnected-(U2-A1-Pad16) -> /A1
- U2 pad 2: unconnected-(U2-GPB1-Pad2) -> Net-(U2-GPB1)
- U2 pad 3: unconnected-(U2-GPB2-Pad3) -> Net-(U2-GPB2)
- U2 pad 9: unconnected-(U2-V_{DD}-Pad9) -> +3V3
Routing:
- net /ROW2: track 0.00 -> 327.3 mm
- net /ROW0: track 285.8 -> 0.00 mm
- net Net-(U2-GPB0): track 0.00 -> 249.5 mm
- net Net-(U2-GPB1): track 0.00 -> 234.4 mm
- net Net-(U2-GPB2): track 0.00 -> 224.4 mm
- net +3V3: track 0.00 -> 184.5 mm
- net /A1: track 0.00 -> 174.6 mm
- net /A0: track 0.00 -> 172.8 mm
- net /ROW5: track 285.6 -> 387.1 mm
- net /COL0: track 85.8 -> 0.00 mm
- net /ROW4: track 275.0 -> 358.2 mm
- net /COL15: track 0.00 -> 76.2 mm
- net /ROW3: track 280.8 -> 345.7 mm
- net /COL11: track 44.0 -> 92.0 mm
- net /COL12: track 84.1 -> 44.0 mm
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
Commit message: pcb export 1 but im gonna change it anyway
help im going to shift the microcontroller up a bit
Parts:
- moved REF** 155.1 mm to (219.3, 25.1), turned to 0 degrees
Connections:
- U2 pad 18: unconnected-(U2-~{RESET}-Pad18) -> +3V3
Routing:
- net +3V3: track 184.5 -> 264.2 mm
